File: Electronics/v0.2/UniversalNode.kicad_pcb (KiCad board)
At the start: 2 copper layers, 134 x 134 mm, 112 parts, among them IC1 HX711, J1 Screw_Terminal_01x02, J10 Screw_Terminal_01x02, J2 Screw_Terminal_01x04, J3 CONUFL001-SMD-T, J4 Screw_Terminal_01x03, J5 Screw_Terminal_01x03, J6 PJ-006A-SMT, J7 Conn_02x03_Top_Bottom, J8 Conn_02x03_Top_Bottom, J9 Screw_Terminal_01x02, Q1 AOD417, Q2 AOD417, Q3 DMG3406L, T1 MMBT4403L, U1 Teensy3.6, U2 FeatherM0_LoRaWAN, U3 LT3652IMSETRPBF, U4 COM-13909, U5 MT3608, U6 MT3608, U7 DW06D

Commit message: finalising version 0.2
Parts:
- removed G*** (x2): LOGO, SilkscreenImages:NSWGov
- removed J10, J9: Screw_Terminal_01x02, TerminalBlock:TerminalBlock_bornier-2_P5.08mm
- removed JP1: Enable Debug, Jumper:SolderJumper-2_P1.3mm_Open_Pad1.0x1.5mm
- removed JP2: Enable SM, Jumper:SolderJumper-2_P1.3mm_Open_Pad1.0x1.5mm
- removed JP3: Enable Weather, Jumper:SolderJumper-2_P1.3mm_Open_Pad1.0x1.5mm
- removed JP4: Enable FeaM0 AGND, Jumper:SolderJumper-2_P1.3mm_Open_Pad1.0x1.5mm
- removed JP5: Enable 9V Control, Jumper:SolderJumper-2_P1.3mm_Open_Pad1.0x1.5mm
- removed JP6: Enable LoRaWAN, Jumper:SolderJumper-2_P1.3mm_Open_Pad1.0x1.5mm
- removed JP7: Enable SCL, Jumper:SolderJumper-2_P1.3mm_Open_Pad1.0x1.5mm
- removed JP8: Enable SDA, Jumper:SolderJumper-2_P1.3mm_Open_Pad1.0x1.5mm
- removed S1: L101011MS02Q, L101011MS02Q:SW_L101011MS02Q
- removed TP1: Bat+, TestPoint:TestPoint_Pad_D2.0mm
- removed TP2: Bat-, TestPoint:TestPoint_Pad_D2.0mm
- added C18: 0.1uF, Capacitor_SMD:C_0805_2012Metric, F.Cu at (153.9, 107.7)
- added C19: 0.1uF, Capacitor_SMD:C_0805_2012Metric, F.Cu at (163.6, 94.6)
- added C20: 0.1uF, Capacitor_SMD:C_0805_2012Metric, F.Cu at (164.1, 111.3)
- added C21: 0.1uF, Capacitor_SMD:C_0805_2012Metric, F.Cu at (185.4, 95.2)
- added C22: 0.1uF, Capacitor_SMD:C_0805_2012Metric, F.Cu at (185.4, 91.7)
- added D13: LED, LED_SMD:LED_0805_2012Metric, F.Cu at (168.9, 94.0)
- added D14: LED, LED_SMD:LED_0805_2012Metric, F.Cu at (146.3, 99.8)
- added D15: LED, LED_SMD:LED_0805_2012Metric, F.Cu at (149.4, 109.0)
- added J11: Conn_01x06_Male, Connector_PinHeader_2.54mm:PinHeader_1x06_P2.54mm_Vertical, F.Cu at (159.3, 110.0)
- added J12: MEM2075-00-140-01-A, MEM2075-00-140-01-A:GCT_MEM2075-00-140-01-A, F.Cu at (137.7, 118.9)
- added R37: 10K, Resistor_SMD:R_0805_2012Metric, F.Cu at (166.1, 96.8)
- added R38: 330, Resistor_SMD:R_0805_2012Metric, F.Cu at (148.8, 102.4)
- added R39: 10K, Resistor_SMD:R_0805_2012Metric, F.Cu at (152.1, 111.8)
- added R40: 1K, Resistor_SMD:R_0805_2012Metric, F.Cu at (147.3, 106.7)
- added R41: 10K, Resistor_SMD:R_0805_2012Metric, F.Cu at (144.3, 104.4)
- added S6: KS11R21CQD, KS11R21CQD:SW_KS11R21CQD, F.Cu at (137.9, 148.1)
- added Y1: 9C-8.000MEEJ-T, 9C-8:XTAL_9C-8.000MEEJ-T, F.Cu at (165.4, 88.6)
- R35: value 10K -> 330
- S2, S4: value L101011MS02Q -> KS11R21CQD; footprint L101011MS02Q:SW_L101011MS02Q -> KS11R21CQD:SW_KS11R21CQD
- S3: value L101011MS02Q -> FSM8JH; footprint L101011MS02Q:SW_L101011MS02Q -> FSM8JH:SW_FSM8JH
- U1: value Teensy3.6 -> ATmega328-AU; footprint teensyBoards:Teensy35_36 -> Package_QFP:TQFP-32_7x7mm_P0.8mm
- U2: value FeatherM0_LoRaWAN -> TPS73633DBVT; footprint FeatherM0:FeatherM0 -> TPS73633DBVT:SOT95P280X145-5N
- moved S2 129.5 mm to (93.3, 102.3)
- moved R12 98.2 mm to (98.0, 115.7), turned to 90 degrees
- moved S4 86.9 mm to (202.7, 117.6)
- moved R13 86.3 mm to (103.6, 47.8)
- moved D4 86.3 mm to (98.6, 47.8)
- moved J7 83.3 mm to (158.8, -40.4)
- moved J8 83.3 mm to (150.4, -40.4)
- moved S3 83.0 mm to (161.3, 117.3), turned to 45 degrees
- moved D5 79.4 mm to (109.6, 56.6)
- moved R14 79.4 mm to (114.6, 56.6)
- moved R23 76.3 mm to (186.2, 112.8)
- moved R21 71.2 mm to (186.3, 109.5), turned to 0 degrees
- moved J4 64.1 mm to (192.3, 107.4)
- moved C14 58.4 mm to (172.2, 115.1), turned to 0 degrees
- moved C13 54.4 mm to (152.9, 127.0)
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Connections:
- C12 pad 2: GNDA -> GND
- C3 pad 2: GNDA -> GND
- C4 pad 2: GNDA -> GND
- C6 pad 2: GNDA -> GND
- IC1 pad 10: GNDA -> GND
- IC1 pad 13: Net-(IC1-Pad13) -> (no net)
- IC1 pad 14: GNDA -> GND
- IC1 pad 5: GNDA -> GND
- IC1 pad 9: GNDA -> GND
- J2 pad 2: GNDA -> GND
- J3 pad 2: GNDA -> GND
- J3 pad 3: GNDA -> GND
- J4 pad 3: GNDA -> /9V_GND
- J5 pad 1: /5V_Teensy -> /5V_OUT
- J5 pad 3: GNDA -> GND
- J6 pad 1: Net-(D8-Pad1) -> Net-(J6-Pad1)
- J7 pad 2: /SDA -> /SCL
- J7 pad 5: /SCL -> /SDA
- J8 pad 2: +3V3 -> GND
- J8 pad 4: GNDA -> GND
- J8 pad 5: GNDA -> +3V3
- J8 pad 6: GNDA -> GND
- JP9 pad 2: GNDA -> GND
- R11 pad 2: GNDA -> GND
- R15 pad 1: /L_CS -> /Lora_CS
- R23 pad 1: GNDA -> /9V_GND
- R24 pad 1: GNDA -> GND
- S2 pad 1: /5V_Teensy -> Net-(R12-Pad2)
- S3 pad 1: Net-(S3-Pad1) -> GND
- S3 pad 2: /5V_OUT -> GND
- S4 pad 1: /Debug -> Net-(D1-Pad1)
- S5 pad 2: Net-(S5-Pad2) -> GND
- S5 pad 4: Net-(S5-Pad4) -> Net-(C17-Pad2)
- U1 pad 1: GND -> /9V_EN
- U1 pad 10: Net-(U1-Pad10) -> /Lora_CS
- U1 pad 11: /Reset -> /G2
- U1 pad 12: /L_CS -> /LoRa_Debug
- U1 pad 13: /MOSI -> /Scale_Debug
- U1 pad 14: /MISO -> /Card_Detect
- U1 pad 15: Net-(U1-Pad15) -> /MOSI
- U1 pad 16: /LoRa_Debug -> /MISO
- U1 pad 17: /Scale_Debug -> /SCK
- U1 pad 18: Net-(U1-Pad18) -> +3V3
- U1 pad 19: Net-(U1-Pad19) -> (no net)
- U1 pad 2: /Debug -> /G0
- U1 pad 21: Net-(U1-Pad21) -> GND
- U1 pad 22: Net-(U1-Pad22) -> (no net)
- U1 pad 23: Net-(U1-Pad23) -> /Weather_Data
- U1 pad 24: Net-(U1-Pad24) -> /SM_Data
- U1 pad 3: Net-(U1-Pad3) -> GND
- U1 pad 30: Net-(U1-Pad30) -> /Rx
- U1 pad 31: Net-(U1-Pad31) -> /Tx
- U1 pad 32: Net-(U1-Pad32) -> /Debug(INT)
- U1 pad 4: /G0 -> +3V3
- U1 pad 5: Net-(U1-Pad5) -> GND
- U1 pad 6: Net-(U1-Pad6) -> +3V3
- U1 pad 7: /G1 -> Net-(U1-Pad7)
- U1 pad 8: /G2 -> Net-(U1-Pad8)
- U1 pad 9: Net-(U1-Pad9) -> /G1
- U3 pad 8: Net-(U3-Pad8) -> (no net)
- U4 pad 1: GNDA -> GND
- U4 pad 10: GNDA -> GND
- U4 pad 11: Net-(U4-Pad11) -> (no net)
- U4 pad 12: Net-(U4-Pad12) -> (no net)
- U4 pad 5: /L_CS -> /Lora_CS
- U4 pad 7: Net-(U4-Pad7) -> (no net)
- U4 pad 8: GNDA -> GND
- U5 pad 6: Net-(U5-Pad6) -> (no net)
- U6 pad 6: Net-(U6-Pad6) -> (no net)
- U7 pad 4: Net-(U7-Pad4) -> (no net)
Routing:
- net +3V3: track 198.0 -> 60.2 mm, vias 6 -> 0
- net Net-(S3-Pad1): track 77.9 -> 0.00 mm, vias 2 -> 0
- net /SM_Data: track 77.6 -> 3.34 mm, vias 6 -> 0
- net /5V_Teensy: track 72.5 -> 0.00 mm, vias 2 -> 0
- net /Scale_Debug: track 72.0 -> 0.00 mm, vias 2 -> 0
- net /Weather_Data: track 72.1 -> 3.30 mm
- net /9V_EN: track 87.5 -> 27.6 mm
- net /V_BAT: track 192.7 -> 132.8 mm, vias 2 -> 4
- net /LoRa_Debug: track 59.1 -> 0.00 mm, vias 1 -> 0
- net /MISO: track 46.9 -> 0.00 mm
- net /Debug: track 45.5 -> 0.00 mm, vias 1 -> 0
- net /SDA: track 110.1 -> 65.3 mm, vias 4 -> 2
- net Net-(JP7-Pad1): track 44.6 -> 0.00 mm
- net /9V_OUT: track 103.3 -> 59.6 mm, vias 4 -> 0
- net Net-(JP8-Pad1): track 40.4 -> 0.00 mm, vias 1 -> 0
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- removed copper zone on B.Cu, net GNDA
- removed copper zone on F.Cu, net GNDA
Other:
- board text added: "5V SDI-12"
- board text added: "9V SDI-12"
- board text added: "Battery ON"
- board text added: "Harvey Bates 05/21"
- board text removed: "3.3V"
- board text removed: "5V"
- board text removed: "5V OUT"
- board text removed: "9V"
- board text removed: "9V OUT"
- board text removed: "AGND"
- board text removed: "Feather"
- board text removed: "GND"
- board text removed: "Harvey Bates 04/21"
- board text removed: "OFF"
- board text removed: "ON"
- board text removed: "SCL"
- board text removed: "SDA"
- board text removed: "Teensy"

Commit message: finalised v0.2
Parts:
- removed D4, D5: LED, LED_SMD:LED_0805_2012Metric
- removed JP9: Scale SPS, Jumper:SolderJumper-2_P1.3mm_Bridged_Pad1.0x1.5mm
- removed R10: 20K, Resistor_SMD:R_0805_2012Metric
- removed R8, R9: 100, Resistor_SMD:R_0805_2012Metric
- removed the REF** at (94.5, 90.0)
- added BT1: BK-18650-PC6, BAT_BK-18650-PC6, B.Cu at (114.6, 114.8)
- added C23: 0.1uF, Capacitor_SMD:C_0805_2012Metric, F.Cu at (179.1, 58.2)
- added C24: 0.1uF, Capacitor_SMD:C_0805_2012Metric, F.Cu at (117.9, 43.7)
- added C25: 0.1uF, Capacitor_SMD:C_0805_2012Metric, F.Cu at (119.4, 73.2)
- added C26: 0.1uF, Capacitor_SMD:C_0805_2012Metric, F.Cu at (172.0, 63.0)
- added C27: 0.1uF, Capacitor_SMD:C_0805_2012Metric, F.Cu at (124.0, 29.5)
- added C28: 0.1uF, Capacitor_SMD:C_0805_2012Metric, F.Cu at (106.7, 68.6)
- added C29: 0.1uF, Capacitor_SMD:C_0805_2012Metric, F.Cu at (186.4, 30.7)
- added C30: 10nF, Capacitor_SMD:C_0805_2012Metric, F.Cu at (113.8, 43.7)
- added C31: 10nF, Capacitor_SMD:C_0805_2012Metric, F.Cu at (126.7, 62.7)
- added C32: 10nF, Capacitor_SMD:C_0805_2012Metric, F.Cu at (185.9, 40.6)
- added C33: 10uF, Capacitor_SMD:CP_Elec_5x5.4, F.Cu at (94.5, 28.2)
- added C34: 10uF, Capacitor_SMD:CP_Elec_5x5.4, F.Cu at (94.2, 52.1)
- added C35: 10uF, Capacitor_SMD:CP_Elec_5x5.4, F.Cu at (194.1, 30.5)
- added C36: 0.1uF, Capacitor_SMD:C_0805_2012Metric, F.Cu at (111.3, 26.4)
- added C37: 0.1uF, Capacitor_SMD:C_0805_2012Metric, F.Cu at (112.3, 60.2)
- added C38: 0.1uF, Capacitor_SMD:C_0805_2012Metric, F.Cu at (182.6, 33.3)
- added C39: 0.1uF, Capacitor_SMD:C_0805_2012Metric, F.Cu at (107.5, 26.4)
- added C40: 0.1uF, Capacitor_SMD:C_0805_2012Metric, F.Cu at (109.3, 61.0)
- added C41: 0.1uF, Capacitor_SMD:C_0805_2012Metric, F.Cu at (178.2, 52.1)
- added D17: LED, LED_SMD:LED_0805_2012Metric, F.Cu at (130.5, 59.3)
- added D18: LED, LED_SMD:LED_0805_2012Metric, F.Cu at (139.7, 72.1)
- added D19: LED, LED_SMD:LED_0805_2012Metric, F.Cu at (180.1, 60.7)
- added G***: LOGO, SilkscreenImages:NSWGov, F.Cu at (114.4, 114.3)
- added IC2: HX711, HX711:SOIC127P600X160-16N, F.Cu at (113.3, 66.5)
- added IC3: HX711, HX711:SOIC127P600X160-16N, F.Cu at (182.1, 46.0)
- added J10: Screw_Terminal_01x04, TerminalBlock:TerminalBlock_bornier-4_P5.08mm, B.Cu at (192.5, 38.4)
- added J9: Screw_Terminal_01x04, TerminalBlock:TerminalBlock_bornier-4_P5.08mm, B.Cu at (102.1, 53.1)
- added JP1: Scale SPS, Jumper:SolderJumper-2_P1.3mm_Bridged_Pad1.0x1.5mm, F.Cu at (121.2, 37.1)
- added JP2: Scale SPS, Jumper:SolderJumper-2_P1.3mm_Bridged_Pad1.0x1.5mm, F.Cu at (119.4, 61.0)
- added JP3: Scale SPS, Jumper:SolderJumper-2_P1.3mm_Bridged_Pad1.0x1.5mm, F.Cu at (182.5, 55.9)
- added R42: 10K, Resistor_SMD:R_0805_2012Metric, F.Cu at (120.7, 68.3)
- added R43: 10K, Resistor_SMD:R_0805_2012Metric, F.Cu at (196.2, 62.7)
- added R44: 100, Resistor_SMD:R_0805_2012Metric, F.Cu at (106.9, 36.6)
- added R45: 100, Resistor_SMD:R_0805_2012Metric, F.Cu at (106.7, 64.8)
- added R46: 100, Resistor_SMD:R_0805_2012Metric, F.Cu at (178.3, 54.4)
- added R47: 100, Resistor_SMD:R_0805_2012Metric, F.Cu at (106.9, 32.8)
- added R48: 100, Resistor_SMD:R_0805_2012Metric, F.Cu at (109.2, 58.7)
- added R49: 100, Resistor_SMD:R_0805_2012Metric, F.Cu at (179.1, 40.0)
- added R50: 20K, Resistor_SMD:R_0805_2012Metric, F.Cu at (118.1, 24.6)
- added R51: 8.2K, Resistor_SMD:R_0805_2012Metric, F.Cu at (118.1, 26.9)
- added R52: 20K, Resistor_SMD:R_0805_2012Metric, F.Cu at (115.4, 61.0)
- added R53: 8.2K, Resistor_SMD:R_0805_2012Metric, F.Cu at (120.8, 65.3)
- added R54: 20K, Resistor_SMD:R_0805_2012Metric, F.Cu at (182.1, 40.6)
- added R55: 8.2K, Resistor_SMD:R_0805_2012Metric, F.Cu at (184.2, 36.8)
- added R56: 10K, Resistor_SMD:R_0805_2012Metric, F.Cu at (120.4, 32.5)
- added R57: 10K, Resistor_SMD:R_0805_2012Metric, F.Cu at (115.4, 57.1)
- added R58: 10K, Resistor_SMD:R_0805_2012Metric, F.Cu at (185.8, 51.6)
- added S1: FSM8JH, FSM8JH:SW_FSM8JH, F.Cu at (110.2, 50.8)
- added S7: FSM8JH, FSM8JH:SW_FSM8JH, F.Cu at (107.4, 83.1)
- added S8: FSM8JH, FSM8JH:SW_FSM8JH, F.Cu at (203.5, 61.7)
- added T2: MMBT4403L, MMBT4403L:SOT23, F.Cu at (122.7, 61.8)
- added T3: MMBT4403L, MMBT4403L:SOT23, F.Cu at (188.2, 34.8)
- added TP1: Bat+, TestPoint:TestPoint_Pad_D2.0mm, B.Cu at (147.6, 126.2)
- added TP2: Bat-, TestPoint:TestPoint_Pad_D2.0mm, B.Cu at (147.6, 130.0)
- added U10: ATmega328-AU, Package_QFP:TQFP-32_7x7mm_P0.8mm, F.Cu at (167.1, 56.4)
- added U8: ATmega328-AU, Package_QFP:TQFP-32_7x7mm_P0.8mm, F.Cu at (121.7, 51.8)
- added U9: ATmega328-AU, Package_QFP:TQFP-32_7x7mm_P0.8mm, F.Cu at (129.3, 71.4)
- added Y2: 9C-8.000MEEJ-T, 9C-8:XTAL_9C-8.000MEEJ-T, F.Cu at (94.2, 65.0)
- added Y3: 9C-8.000MEEJ-T, 9C-8:XTAL_9C-8.000MEEJ-T, F.Cu at (124.2, 82.5)
- added Y4: 9C-8.000MEEJ-T, 9C-8:XTAL_9C-8.000MEEJ-T, F.Cu at (173.5, 44.2)
- C4: value 10nF -> 0.1uF
- C6: value 10uF -> 0.1uF; footprint Capacitor_SMD:CP_Elec_5x5.4 -> Capacitor_SMD:C_0805_2012Metric
- D1, D11, D12, D15, D2, D3, J1, J11, J12, J3, J4, J5, R1, R3, R34, R35, R4, S2, S3, S4, S5, S6: moved to B.Cu
- J2: value Screw_Terminal_01x04 -> Conn_01x06_Male; footprint TerminalBlock:TerminalBlock_bornier-4_P5.08mm -> Connector_PinHeader_2.54mm:PinHeader_1x06_P2.54mm_Vertical; moved to B.Cu
- J6: value PJ-006A-SMT -> Conn_01x06_Male; footprint PJ-006A-SMT:CUI_PJ-006A-SMT -> Connector_PinHeader_2.54mm:PinHeader_1x06_P2.54mm_Vertical; moved to B.Cu
- J7: value Conn_02x03_Top_Bottom -> Conn_01x06_Male; footprint Connector_PinHeader_2.54mm:PinHeader_2x03_P2.54mm_Vertical -> Connector_PinHeader_2.54mm:PinHeader_1x06_P2.54mm_Vertical; moved to B.Cu
- J8: value Conn_02x03_Top_Bottom -> Screw_Terminal_01x04; footprint Connector_PinHeader_2.54mm:PinHeader_2x03_P2.54mm_Vertical -> TerminalBlock:TerminalBlock_bornier-4_P5.08mm; moved to B.Cu
- R11: value 8.2K -> 330
- R13, R14: value 220 -> 330
- moved R12 114.2 mm to (179.1, 35.3)
- moved S2 107.8 mm to (174.3, 31.2), turned to 270 degrees
- moved J7 102.9 mm to (184.9, 59.2), turned to 270 degrees
- moved J2 102.1 mm to (122.7, 40.6), turned to 90 degrees
- moved T1 96.8 mm to (122.7, 25.7), turned to 270 degrees
- moved IC1 91.5 mm to (113.5, 32.5), turned to 270 degrees
- moved C3 88.5 mm to (127.5, 47.2), turned to 180 degrees
- moved J8 84.7 mm to (102.1, 29.2), turned to 270 degrees
- moved C7 84.3 mm to (125.0, 44.2)
- moved S3 82.0 mm to (162.3, 35.3), turned to 0 degrees
- moved R11 77.0 mm to (127.8, 56.6), turned to 135 degrees
- moved R25 74.0 mm to (109.9, 43.7), turned to 180 degrees
- moved C6 73.1 mm to (160.3, 60.5), turned to 225 degrees
- moved J6 71.4 mm to (114.0, 73.4), turned to 90 degrees
- moved C20 71.2 mm to (167.9, 40.1), turned to 90 degrees
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Connections:
- C17 pad 2: Net-(C17-Pad2) -> Net-(BT1-Pad1)
- C4 pad 1: +3V3 -> Net-(C4-Pad1)
- C6 pad 1: Net-(C3-Pad1) -> Net-(C6-Pad1)
- C7 pad 1: Net-(C7-Pad1) -> +3V3
- C7 pad 2: Net-(C7-Pad2) -> GND
- C9 pad 1: Net-(C9-Pad1) -> +3V3
- C9 pad 2: Net-(C9-Pad2) -> GND
- IC1 pad 11: /SCL -> /1_SCL
- IC1 pad 12: /SDA -> /1_SDA
- IC1 pad 3: Net-(C3-Pad1) -> Net-(C27-Pad1)
- IC1 pad 4: Net-(C7-Pad2) -> Net-(C36-Pad2)
- IC1 pad 6: Net-(C7-Pad1) -> Net-(C36-Pad1)
- IC1 pad 7: Net-(C9-Pad1) -> Net-(C39-Pad1)
- IC1 pad 8: Net-(C9-Pad2) -> Net-(C39-Pad2)
- J2 pad 1: Net-(C3-Pad1) -> /1_DTR
- J2 pad 2: GND -> /1_Rx
- J2 pad 3: Net-(J2-Pad3) -> /1_Tx
- J2 pad 4: Net-(J2-Pad4) -> +3V3
- J6 pad 1: Net-(J6-Pad1) -> /2_DTR
- J6 pad 2: Net-(C17-Pad2) -> /2_Rx
- J6 pad 3: Net-(C17-Pad2) -> /2_Tx
- J7 pad 1: /SDA -> /3_DTR
- J7 pad 2: /SCL -> /3_Rx
- J7 pad 3: /SDA -> /3_Tx
- J7 pad 4: /SCL -> +3V3
- J7 pad 5: /SDA -> GND
- J7 pad 6: /SCL -> GND
- J8 pad 1: +3V3 -> Net-(C27-Pad1)
- J8 pad 3: +3V3 -> Net-(J8-Pad3)
- J8 pad 4: GND -> Net-(J8-Pad4)
- R11 pad 1: Net-(C7-Pad2) -> Net-(D17-Pad2)
- R11 pad 2: GND -> /1_SCK
- R13 pad 2: GND -> /2_SCK
- R14 pad 2: GND -> /3_SCK
- R25 pad 2: Net-(IC1-Pad15) -> /1_Reset
- R27 pad 2: Net-(C17-Pad2) -> Net-(BT1-Pad1)
- S5 pad 3: Net-(C17-Pad2) -> Net-(BT1-Pad1)
- S5 pad 4: Net-(C17-Pad2) -> Net-(BT1-Pad1)
- S6 pad 3: Net-(J6-Pad1) -> Net-(BT1-Pad3+)
- T1 pad 3: Net-(C3-Pad1) -> Net-(C27-Pad1)
- U1 pad 12: /LoRa_Debug -> (no net)
- U1 pad 13: /Scale_Debug -> (no net)
- U7 pad 3: Net-(C17-Pad2) -> Net-(BT1-Pad1)
- U7 pad 6: Net-(C17-Pad2) -> Net-(BT1-Pad1)
Routing:
- net +3V3: track 60.2 -> 431.9 mm, vias 0 -> 21
- net Net-(BT1-Pad1): track 0.00 -> 112.6 mm
- net /9V_EN: track 27.6 -> 109.1 mm, vias 2 -> 6
- net /SM_Data: track 3.34 -> 75.4 mm, vias 0 -> 4
- net Net-(C28-Pad1): track 0.00 -> 67.4 mm, vias 0 -> 3
- net Net-(C17-Pad2): track 65.5 -> 0.00 mm
- net Net-(BT1-Pad3+): track 0.00 -> 59.4 mm
- net /MISO: track 0.00 -> 56.2 mm, vias 0 -> 1
- net GND: track 17.3 -> 64.4 mm, vias 13 -> 45
- net /MOSI: track 20.4 -> 65.0 mm, vias 2 -> 3
- net /Card_Detect: track 3.60 -> 48.1 mm, vias 0 -> 3
- net Net-(C27-Pad1): track 0.00 -> 43.1 mm, vias 0 -> 1
- net /3_Reset: track 0.00 -> 42.6 mm
- net /Weather_Data: track 3.30 -> 45.3 mm, vias 0 -> 4
- net /SCK: track 23.6 -> 64.8 mm, vias 0 -> 2
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Other:
- board text added: "ANT"
- board text added: "Batt (+)"
- board text added: "Batt (-)"
- board text added: "Battery On/Off"
- board text added: "Debug Mode On/Off"
- board text added: "GND"
- board text added: "MC-1 TTL"
- board text added: "MC-2 TTL"
- board text added: "MC-3 TTL"
- board text added: "MC-Master TTL"
- board text added: "RST"
- board text added: "SD-Card Logger"
- board text added: "Solar On/Off"
- board text added: "WeighScale One"
- board text added: "WeighScale Three"
- board text added: "WeighScale Two"
- board text removed: "Closed: 10 Hz Open: 80 Hz"
- board text removed: "DEBUG MODE"
- board text removed: "LoRa Active"
- board text removed: "SOLAR"
- board text removed: "Scale Active"
- board text removed: "WEIGHSCALE"
