File: Electronics/v0.3/UniversalNode.kicad_pcb (KiCad board)
At the start: 2 copper layers, 134 x 134 mm, 157 parts, among them IC1 HX711, IC2 HX711, IC3 HX711, J1 Screw_Terminal_01x02, J10 Screw_Terminal_01x04, J2 Conn_01x06_Male, J3 CONUFL001-SMD-T, J4 Screw_Terminal_01x03, J5 Screw_Terminal_01x03, J6 Conn_01x06_Male, J7 Conn_01x06_Male, J8 Screw_Terminal_01x04, J9 Screw_Terminal_01x04, Q1 AOD417, Q2 AOD417, Q3 DMG3406L, T1 MMBT4403L, T2 MMBT4403L, T3 MMBT4403L, U1 Teensy3.6, U10 ATmega328-AU, U3 LT3652IMSETRPBF, U4 COM-13909, U5 MT3608, U6 MT3608, U7 DW06D, U8 ATmega328-AU, U9 ATmega328-AU, Y2 9C-8.000MEEJ-T, Y3 9C-8.000MEEJ-T, Y4 9C-8.000MEEJ-T

Commit message: updated v0.3 and sent for production
Parts:
- added G***: LOGO, SilkscreenImages:NSWGov, F.Cu at (114.6, 105.7)
- moved TP2 87.7 mm to (90.4, 72.6), turned to 0 degrees
- moved TP1 87.5 mm to (86.9, 72.6), turned to 0 degrees
- moved Y2 30.4 mm to (114.3, 48.3)
- moved R43 25.5 mm to (173.2, 37.8)
- moved R9 22.4 mm to (136.1, 57.9), turned to 45 degrees
- moved C28 16.1 mm to (123.6, 53.6), turned to 0 degrees
- moved R10 13.4 mm to (186.5, 54.6), turned to 180 degrees
- moved C30 7.25 mm to (122.7, 31.8)
- moved C27 7.08 mm to (126.0, 25.7)
- moved C39 6.38 mm to (108.0, 35.3), turned to 90 degrees
- moved R51 6.32 mm to (113.9, 25.9), turned to 180 degrees
- moved C40 6.18 mm to (108.2, 60.2), turned to 270 degrees
- moved R48 4.88 mm to (108.2, 56.4), turned to 90 degrees
- moved R47 4.06 mm to (108.0, 31.2)
- moved JP2 3.16 mm to (116.5, 66.0), turned to 180 degrees
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Routing:
- net /3.3_1: track 0.00 -> 114.4 mm, vias 0 -> 5
- net /3.3_3: track 0.00 -> 114.2 mm, vias 0 -> 3
- net /SCL: track 2.81 -> 114.4 mm, vias 0 -> 6
- net /SDA: track 3.72 -> 113.9 mm, vias 0 -> 5
- net /3.3_2: track 0.00 -> 100.6 mm, vias 0 -> 1
- net /INT_Teensy3: track 0.00 -> 90.8 mm, vias 0 -> 7
- net GND: track 10.3 -> 70.2 mm, vias 14 -> 98
- net Net-(BT1-Pad1+): track 114.2 -> 58.9 mm
- net Net-(C28-Pad1): track 0.00 -> 49.0 mm
- net /INT_Teensy1: track 0.00 -> 46.8 mm, vias 0 -> 2
- net Net-(C27-Pad1): track 0.00 -> 44.5 mm
- net /3_Reset: track 0.00 -> 39.9 mm, vias 0 -> 3
- net /2_SCL: track 0.00 -> 36.8 mm, vias 0 -> 2
- net Net-(C29-Pad1): track 0.00 -> 35.2 mm
- net /3_Tx: track 0.00 -> 34.4 mm, vias 0 -> 1
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Other:
- board text added: "AgU-Node"
- board text added: "Universal Node for Agricultural Applications"
