File: electronics/schematics-pcb/UniversalNode.kicad_pcb (KiCad board)
At the start: 2 copper layers, 121.5 x 127.9 mm, 83 parts, among them IC1 HX711, IC2 HX711, IC3 HX711, J1 Screw_Terminal_01x04, J10 Bat_Conn, J11 TBP02R2-381-03BE, J12 TBP02R2-381-03BE, J13 TBP02R2-381-03BE, J14 TBP02R2-381-03BE, J2 Screw_Terminal_01x04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

Commit message: prepared final figures (schematic and pcb) for sup material
Other:
- board text added: "v0.5 by Harvey Bates @ NSW Department of Primary Industries"
- board text removed: "v0.5 by Harvey Bates"
