File: electronics/schematics-pcb/UniversalNode.sch (KiCad schematic (older format))
At the start: 81 parts, among them IC1 HX711, IC2 HX711, IC3 HX711, J1 Screw_Terminal_01x04, J10 Bat_Conn, J11 TBP02R2-381-03BE, J12 TBP02R2-381-03BE, J13 TBP02R2-381-03BE, J14 TBP02R2-381-03BE, J15 Bat_Conn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

Commit message: prepared final figures (schematic and pcb) for sup material
Parts:
- removed BT1: BK-18650-PC6, BK-18650-PC6:BAT_BK-18650-PC6, symbol BK-18650-PC6:BK-18650-PC6
- removed J15: Bat_Conn, TerminalBlock:102-6492-ND‎, symbol TBP02R2-381-02BE:TBP02R2-381-02BE
Connections:
- wire segments 207 -> 199
Other:
- note added: "- Harvey Bates @ NSW Department of Primary Industries"
- note added: "12th April 2022"
- note added: "ACD (Weigh-station)"
- note added: "Ag-Node"
- note removed: "- Harvey Bates"
- note removed: "7th August 2021"
- note removed: "AgU-Node"
- note removed: "HX711 (WeighScale)"
- moved on the sheet: J10, J11, J12, J13, J14, J5, J7, J8, R43, U2
